File: Schematics and Manuals/Reverse Engineering/REG04/REG04.kicad_sch (KiCad schematic)
At the start: 30 parts, among them J1 Conn_01x40, Q1 PNP, Q11 PNP, Q3 PNP

Commit message: Added my notes on bruce273's reverse Engineered version of the REC04 PCB and an analog way to test the cards 8 lines at a time
Parts:
- removed D1, D2: 4.3V, symbol Device:D_Zener
- removed D51, D52, D53, D54, D55, D56, D57, D58, D59, D60: D, symbol Device:D
- removed J1: Conn_01x40, symbol Connector_Generic:Conn_01x40
- removed Q1, Q11, Q3: PNP, symbol Simulation_SPICE:PNP
- added C10, C11, C12, C16, C17, C18, C19, C20, C3, C4, C5, C6, C7, C8, C9: C, Capacitor_THT:C_Rect_L7.0mm_W2.0mm_P5.00mm, symbol Device:C
- added C21: C, Capacitor_THT:C_Axial_L12.0mm_D6.5mm_P15.00mm_Horizontal, symbol Device:C
- added C22: C, Capacitor_THT:C_Axial_L5.1mm_D3.1mm_P12.50mm_Horizontal, symbol Device:C
- added C23: 2.2, Capacitor_THT:C_Axial_L5.1mm_D3.1mm_P12.50mm_Horizontal, symbol Device:C
- added D1, D10, D11, D12, D13, D14, D15, D16, D17, D18, D19, D2, D20, D21, D22, D23, D24, D25, D26, D27, D28, D29, D3, D30, D31, D32, D33, D34, D35, D36, D37, D38, D39, D4, D40, D41, D42, D46, D47, D5, D6, D7, D8, D9: 1N4148, Diode_THT:D_A-405_P12.70mm_Horizontal, symbol Diode:1N4148
- added D43, D44, D45, D48: D_Zener, Diode_THT:D_A-405_P12.70mm_Horizontal, symbol Device:D_Zener
- added J1, J10, J11, J12, J13, J14, J15, J16, J17, J18, J19, J2, J20, J21, J22, J23, J24, J25, J26, J27, J28, J29, J3, J30, J31, J32, J33, J34, J35, J36, J37, J38, J39, J4, J40, J5, J6, J7, J8, J9: Conn_01x02_Pin, TestPoint:TestPoint_2Pads_Pitch5.08mm_Drill1.3mm, symbol Connector:Conn_01x02_Pin
- added Q1, Q10, Q11, Q12, Q13, Q14, Q15, Q16, Q2, Q3, Q4, Q5, Q6, Q7, Q8, Q9: Q_PNP_EBC, Package_TO_SOT_THT:TO-5-3, symbol Device:Q_PNP_EBC
- added R1, R10, R11, R17, R21, R22, R25, R26, R37, R40, R41, R47, R51, R52, R55, R56, R61, R62, R63, R69, R70, R8, R9: 5k1, custom:R_Axial_DIN0207_L6.3mm_D2.5mm_P12.7 mm_Horizontal, symbol Device:R
- added R12, R13, R23, R38, R43, R53, R58: 510, custom:R_Axial_DIN0207_L6.3mm_D2.5mm_P12.7 mm_Horizontal, symbol Device:R
- added R14, R15, R24, R39, R46, R54, R64, R76: 10k, custom:R_Axial_DIN0207_L6.3mm_D2.5mm_P12.7 mm_Horizontal, symbol Device:R
- added R16: R, custom:R_Axial_DIN0207_L6.3mm_D2.5mm_P12.7 mm_Horizontal, symbol Device:R
- added R18, R45, R48, R6, R60, R7: 3k, custom:R_Axial_DIN0207_L6.3mm_D2.5mm_P12.7 mm_Horizontal, symbol Device:R
- added R19, R2, R44, R49, R5, R59: 2k, custom:R_Axial_DIN0207_L6.3mm_D2.5mm_P12.7 mm_Horizontal, symbol Device:R
- added R20, R27, R3, R4, R42, R50, R57: 39k, custom:R_Axial_DIN0207_L6.3mm_D2.5mm_P12.7 mm_Horizontal, symbol Device:R
- added R65, R66: 1k, custom:R_Axial_DIN0207_L6.3mm_D2.5mm_P12.7 mm_Horizontal, symbol Device:R
- added R67, R74: 1k, Resistor_THT:R_Axial_DIN0207_L6.3mm_D2.5mm_P10.16mm_Horizontal, symbol Device:R
- added R68: 10k, Resistor_THT:R_Axial_DIN0207_L6.3mm_D2.5mm_P10.16mm_Horizontal, symbol Device:R
- added R71: 5k1, Resistor_THT:R_Axial_DIN0207_L6.3mm_D2.5mm_P10.16mm_Horizontal, symbol Device:R
- added R72, R73: 39K, Resistor_THT:R_Axial_DIN0207_L6.3mm_D2.5mm_P10.16mm_Horizontal, symbol Device:R
- added R75: 39K, custom:R_Axial_DIN0207_L6.3mm_D2.5mm_P12.7 mm_Horizontal, symbol Device:R
- C1: value .01uF -> C; footprint (none) -> Capacitor_THT:C_Rect_L7.0mm_W2.0mm_P5.00mm
- C13, C14, C15: value 75pF -> C; footprint (none) -> Capacitor_THT:C_Rect_L7.0mm_W2.0mm_P5.00mm
- C2: value .068uF 150V -> C; footprint (none) -> Capacitor_THT:C_Rect_L7.0mm_W2.0mm_P5.00mm
- R28: value 5.1k -> 510; footprint (none) -> custom:R_Axial_DIN0207_L6.3mm_D2.5mm_P12.7 mm_Horizontal
- R29: value 39k -> 2k; footprint (none) -> custom:R_Axial_DIN0207_L6.3mm_D2.5mm_P12.7 mm_Horizontal
- R30: value 39k -> 3k; footprint (none) -> custom:R_Axial_DIN0207_L6.3mm_D2.5mm_P12.7 mm_Horizontal
- R31: value 5.1k -> R; footprint (none) -> custom:R_Axial_DIN0207_L6.3mm_D2.5mm_P12.7 mm_Horizontal
- R32: value 1k -> 5k1; footprint (none) -> custom:R_Axial_DIN0207_L6.3mm_D2.5mm_P12.7 mm_Horizontal
- R33: value 1k -> 3k; footprint (none) -> custom:R_Axial_DIN0207_L6.3mm_D2.5mm_P12.7 mm_Horizontal
- R34: value 10k -> 2k; footprint (none) -> custom:R_Axial_DIN0207_L6.3mm_D2.5mm_P12.7 mm_Horizontal
- R35: value 5.1k -> 39k; footprint (none) -> custom:R_Axial_DIN0207_L6.3mm_D2.5mm_P12.7 mm_Horizontal
- R36: value 39k -> 5k1; footprint (none) -> custom:R_Axial_DIN0207_L6.3mm_D2.5mm_P12.7 mm_Horizontal
Connections:
- net J1-7 is gone; now on an unnamed net: R34.2
- net +6V: now also R35.1, C21.2, J39.1 (Pin_1), J39.2 (Pin_2), R20.1, R27.1, R3.1, R4.1, R42.1, R50.1, R57.1, R64.2, R72.2, R73.2, R75.2; no longer C1.2, R29.2, R30.2, R36.2
- net -12V: now also R29.1, R34.1, C22.2, J40.1 (Pin_1), J40.2 (Pin_2), R1.1, R10.1, R11.2, R15.1, R17.1, R19.1, R2.1, R22.1, R24.1, R25.2, R37.1, R39.1, R40.2, R44.1, R47.1, R49.1, R5.1, R52.1, R54.1, R55.2, R59.1, R61.2, R62.2, R65.2, R66.2, R67.2, R68.2, R69.2, R70.2, R71.1, R74.2; no longer C2.1, R28.1, R31.1, R33.1, R35.1
- net GND: now also R30.2, R33.2, C21.1, C22.1, C23.2, D12.2 (A), D20.2 (A), D28.2 (A), D3.2 (A), D33.2 (A), J10.1 (Pin_1), J10.2 (Pin_2), J17.1 (Pin_1), J17.2 (Pin_2), J23.1 (Pin_1), J23.2 (Pin_2), J28.1 (Pin_1), J28.2 (Pin_2), J38.1 (Pin_1), J38.2 (Pin_2), J4.1 (Pin_1), J4.2 (Pin_2), Q1.1 (E), Q11.1 (E), Q12.1 (E), Q13.1 (E), Q14.1 (E), Q15.1 (E), Q16.1 (E), Q2.1 (E), Q5.1 (E), Q6.1 (E), Q8.1 (E), Q9.1 (E), R18.2, R45.2, R48.2, R6.2, R60.2, R63.1, R7.2; no longer C1.1, C2.2
- net at R31.2: now also R33.1, C11.1, D18.2 (A), Q8.3 (C), R41.1; no longer C14.2
- net at C13.1: now also D27.1 (K), Q11.2 (B), R50.2, R51.1; no longer R29.1
- net at C13.2: now also D31.1 (K), Q12.3 (C), R51.2, R59.2, R60.1; no longer R28.2
- net at R35.2: now also R36.1, C9.1, D19.1 (K), Q8.2 (B); no longer C15.2
- net at R30.1: now also R29.2, C5.2, D15.1 (K), Q6.3 (C), R21.2; no longer C14.1
- net at C15.1: now also D26.2 (A), Q11.3 (C), R46.2, R48.1, R49.2, R56.1; no longer R36.1
- net J1-10: no longer names the net of R32.2
- net J1-10: now also D17.1 (K), D18.1 (K), Q7.2 (B)
- removed net J1-9: R33.2, R34.1
- new net: C9.2, D23.1 (K), D40.2 (A), Q9.3 (C), R36.2, R44.2, R45.1
- new net: C15.2, D30.1 (K), Q12.2 (B), R56.2, R57.2
- new net: C2.1, D5.1 (K), Q1.2 (B), R3.2, R8.1
- new net: C1.1, D4.2 (A), Q1.3 (C), R14.2, R2.2, R6.1, R9.1
- new net: C11.2, D22.1 (K), Q9.2 (B), R41.2, R42.2
- new net: C7.1, D10.2 (A), Q5.3 (C), R16.2, R18.1, R19.2, R26.1
- new net: C8.2, D14.2 (A), R25.1, R28.1
- new net: D10.1 (K), D9.1 (K), Q4.2 (B), R17.2
- new net: C12.2, D22.2 (A), R40.1, R43.1
- new net: C7.2, D14.1 (K), Q6.2 (B), R26.2, R27.2
- new net: C6.2, D11.2 (A), R22.2, R23.1
- new net: D25.1 (K), D26.1 (K), Q10.2 (B), R47.2
- new net: D38.1 (K), D39.2 (A)
- new net: D33.1 (K), D38.2 (A)
- new net: C2.2, D8.1 (K), Q2.3 (C), R5.2, R7.1, R8.2
- new net: C14.2, D27.2 (A), R52.2, R53.1
- new net: D29.1 (K), R53.2
- new net: C18.1, D34.1 (K), D43.2 (A), D46.1 (K), R71.2
- new net: C4.2, D7.2 (A), R11.1, R13.1
- new net: C20.1, D35.1 (K), D47.1 (K), D48.2 (A), R70.1
- new net: C20.2, D48.1 (K), Q15.2 (B), R75.1
- new net: D21.1 (K), R38.2
- new net: D16.1 (K), R28.2
- new net: D6.1 (K), R13.2
- new net: C16.2, D30.2 (A), R55.1, R58.1
- new net: D32.1 (K), R58.2
- new net: C19.2, D36.1 (K), D37.1 (K), D45.2 (A), R69.1
- new net: C18.2, D43.1 (K), Q14.2 (B), R72.1
- new net: C5.1, D11.1 (K), Q5.2 (B), R20.2, R21.1
- new net: C3.2, D5.2 (A), R10.2, R12.1
- new net: D2.1 (K), R12.2
- new net: C1.2, D7.1 (K), Q2.2 (B), R4.2, R9.2
- new net: J11.1 (Pin_1), J11.2 (Pin_2)
- new net: C17.2, D44.1 (K), Q13.2 (B), R64.1
- new net: D41.2 (A), D44.2 (A)
- new net: C10.2, D19.2 (A), R37.2, R38.1
- new net: C19.1, D45.1 (K), Q16.2 (B), R73.1
- new net: D24.1 (K), R43.2
- new net: D13.1 (K), R23.2
- new net: D1.1 (K), D4.1 (K), Q3.2 (B), R1.2
- new net: J25.1 (Pin_1), J25.2 (Pin_2)
- new net: J13.1 (Pin_1), J13.2 (Pin_2)
- new net: J8.1 (Pin_1), J8.2 (Pin_2)
- new net -2V5: C23.1, D39.1 (K), Q10.1 (E), Q3.1 (E), Q4.1 (E), Q7.1 (E), R61.1
- new net P1: D1.2 (A), J1.1 (Pin_1), J1.2 (Pin_2)
- new net P12: D15.2 (A), J12.1 (Pin_1), J12.2 (Pin_2), R24.2
- new net P14: D17.2 (A), J14.1 (Pin_1), J14.2 (Pin_2)
- new net P15: J15.1 (Pin_1), J15.2 (Pin_2), R31.1
- new net P16 -1V: C10.1, C12.1, D20.1 (K), J16.1 (Pin_1), J16.2 (Pin_2)
- new net P18: D23.2 (A), J18.1 (Pin_1), J18.2 (Pin_2), R39.2
- new net P19: D25.2 (A), J19.1 (Pin_1), J19.2 (Pin_2)
- new net P2: J2.1 (Pin_1), J2.2 (Pin_2), R14.1
- new net P20: J20.1 (Pin_1), J20.2 (Pin_2), R46.1
- new net P21 GRset: D13.2 (A), D2.2 (A), D21.2 (A), D29.2 (A), J21.1 (Pin_1), J21.2 (Pin_2)
- new net P22 -1V: C14.1, C16.1, D28.1 (K), J22.1 (Pin_1), J22.2 (Pin_2)
- new net P24: D31.2 (A), J24.1 (Pin_1), J24.2 (Pin_2), R54.2
- new net P26 Gset: D16.2 (A), D24.2 (A), D32.2 (A), D6.2 (A), J26.1 (Pin_1), J26.2 (Pin_2)
- new net P27: D40.1 (K), J27.1 (Pin_1), J27.2 (Pin_2), R62.1, R63.2
- new net P29 Gout: J29.1 (Pin_1), J29.2 (Pin_2), Q13.3 (C), R65.1
- new net P3 -1V: C3.1, C4.1, D3.1 (K), J3.1 (Pin_1), J3.2 (Pin_2)
- new net P30 A: D42.2 (A), J30.1 (Pin_1), J30.2 (Pin_2), R68.1
- new net P31 IO: D42.1 (K), D47.2 (A), J31.1 (Pin_1), J31.2 (Pin_2), Q14.3 (C), R67.1
- new net P32 Out: D46.2 (A), J32.1 (Pin_1), J32.2 (Pin_2), Q15.3 (C), Q16.3 (C), R74.1, R76.2
- new net P33 B: D34.2 (A), J33.1 (Pin_1), J33.2 (Pin_2)
- new net P34 OutZ: J34.1 (Pin_1), J34.2 (Pin_2), R76.1
- new net P35 C: D35.2 (A), J35.1 (Pin_1), J35.2 (Pin_2)
- new net P36 D: D36.2 (A), J36.1 (Pin_1), J36.2 (Pin_2)
- new net P37 E: D37.2 (A), J37.1 (Pin_1), J37.2 (Pin_2)
- new net P5: D8.2 (A), J5.1 (Pin_1), J5.2 (Pin_2), R15.2
- new net P6: D9.2 (A), J6.1 (Pin_1), J6.2 (Pin_2)
- new net P7: J7.1 (Pin_1), J7.2 (Pin_2), R16.1
- new net P9 -1V: C6.1, C8.1, D12.1 (K), J9.1 (Pin_1), J9.2 (Pin_2)
- new net ~{Gout}: C17.1, D41.1 (K), Q10.3 (C), Q3.3 (C), Q4.3 (C), Q7.3 (C), R66.1
- no-connect marks 0 -> 4
Other:
- note added: "-1V"
- note added: "1"
- note added: "10"
- note added: "11"
- note added: "12"
- note added: "13"
- note added: "14"
- note added: "15"
- note added: "16"
- note added: "17"
- note added: "18"
- note added: "19"
- note added: "2"
- note added: "20"
- note added: "21"
- note added: "22"
- note added: "23"
- note added: "24"
- note added: "25"
- note added: "26"
- note added: "27"
- note added: "28"
- note added: "29"
- note added: "3"
- note added: "30"
- note added: "31"
- note added: "32"
- note added: "33"
- note added: "34"
- note added: "35"
- note added: "36"
- note added: "37"
- note added: "38"
- note added: "39"
- note added: "4"
- note added: "40"
- note added: "5"
- note added: "6"
- note added: "7"
- note added: "8"
- note added: "9"
- note added: "A"
- note added: "B"
- note added: "C"
- note added: "D"
- note added: "E"
- note added: "GOut"
- note added: "GRset"
- note added: "GSet"
- note added: "IO"
- note added: "Minor Edits by Roy20100"
- note added: "Out"
- note added: "OutZ"
- note added: "P32=~{P31&P35}&~{P36&P37} P31=~{P32&P33}&P30"
- note added: "Q3"
- note added: "RE by bruce273"
- note added: "REC04"
- note added: "S1"
- note added: "S2"
- note added: "S3"
- note added: "S4"
- note added: "~{Q}1"
- note added: "~{Q}1 en Gout"
- note added: "~{Q}2"
- note added: "~{Q}2 en Gout"
- note added: "~{Q}3"
- note added: "~{Q}3 en Gout"
- note added: "~{Q}4"
- note added: "~{Q}4 en Gout"
- note removed: "All transistors are 2N964 Germanium PNP, 15V 0.1A Metal tab indicates pin 1 which is emitter Case is electrically connected with pin 3 which is collector Pin 2 is the base All diodes are ???? Germanium"

Commit message: Fixed fixed shape of the independent Flip-Flop in REC04
Connections:
- net GND: now also D12.1 (K), D20.1 (K), D28.1 (K), D3.1 (K); no longer D12.2 (A), D20.2 (A), D28.2 (A), D3.2 (A)
- net at D35.1 (K), D47.1 (K), D48.2 (A)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: now also C20.2; no longer C20.1
- net at D48.1 (K), Q15.2 (B), R75.1: now also C20.1; no longer C20.2
- net P16 -1V renamed P16 Q3-CLK
- net P16 Q3-CLK: now also D20.2 (A); no longer D20.1 (K)
- net P22 -1V renamed P22 Q4-CLK
- net P22 Q4-CLK: now also D28.2 (A); no longer D28.1 (K)
- net P3 -1V renamed P3 Q1-CLK
- net P3 Q1-CLK: now also D3.2 (A); no longer D3.1 (K)
- net P9 -1V renamed P9 Q2-CLK
- net P9 Q2-CLK: now also D12.2 (A); no longer D12.1 (K)
Other:
- note added: "Out=~{IO&C}&~{D&E} IO=~{Out&B}&A"
- moved on the sheet: C18, C19, C20, D12, D20, D28, D3, D34, D35, D36, D37, D42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
