File: Schematics/Reverse Engineering/LD312-1/LD312-1.kicad_sch (KiCad schematic)
At the start: 137 parts, among them J1 Conn_01x40, Q1 PNP, Q10 PNP, Q11 PNP, Q12 PNP, Q13 PNP, Q14 PNP, Q15 PNP, Q16 PNP, Q2 PNP, Q5 PNP, Q6 PNP, Q7 PNP, Q8 PNP, Q9 PNP

Commit message: 2025/8/2
Parts:
- R14, R17, R2, R20, R23, R26, R29, R32, R35, R38, R41, R48, R5: value 18k -> 16k
Changed lines of the file:
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@@
 			)
 		)
-		(property "Value" "18k"
+		(property "Value" "16k"
 			(at 254 98.298 90)
 			(effects
@@
 			)
 		)
-		(property "Value" "18k"
+		(property "Value" "16k"
 			(at 184.15 98.298 90)
 			(effects
@@
 			)
 		)
-		(property "Value" "18k"
+		(property "Value" "16k"
 			(at 185.42 44.958 90)
 			(effects
@@
 			)
 		)
-		(property "Value" "18k"
+		(property "Value" "16k"
 			(at 116.84 44.958 90)
 			(effects
@@
 			)
 		)
-		(property "Value" "18k"
+		(property "Value" "16k"
 			(at 118.11 98.298 90)
 			(effects
@@
 			)
 		)
-		(property "Value" "18k"
+		(property "Value" "16k"
 			(at 321.31 150.368 90)
 			(effects
@@
 			)
 		)
-		(property "Value" "18k"
+		(property "Value" "16k"
 			(at 321.31 98.298 90)
 			(effects
@@
 			)
 		)
-		(property "Value" "18k"
+		(property "Value" "16k"
 			(at 322.58 47.498 90)
 			(effects
@@
 			)
 		)
-		(property "Value" "18k"
+		(property "Value" "16k"
 			(at 254 150.368 90)
 			(effects
@@
 			)
 		)
-		(property "Value" "18k"
+		(property "Value" "16k"
 			(at 184.15 150.368 90)
 			(effects
@@
 			)
 		)
-		(property "Value" "18k"
+		(property "Value" "16k"
 			(at 260.35 203.708 90)
 			(effects
@@
 			)
 		)
-		(property "Value" "18k"
+		(property "Value" "16k"
 			(at 118.11 150.368 90)
 			(effects
@@
 			)
 		)
-		(property "Value" "18k"
+		(property "Value" "16k"
 			(at 254 46.228 90)
 			(effects
