File: Schematics/Reverse Engineering/PA24/PA24.kicad_sch (KiCad schematic)
At the start: 97 parts, among them J1 Conn_01x40, Q1 1N1304, Q10 PNP_G, Q11 NPN?, Q12 PNP_G, Q13 NPN?, Q14 PNP_G, Q15 NPN?, Q16 PNP_G, Q17 NPN?, Q2 PNP_G, Q3 NPN?, Q4 PNP_G, Q5 NPN?, Q6 PNP_G, Q7 NPN?, Q8 PNP_G, Q9 NPN?

Commit message: fixed wrong internal power rail from -3.3 to -9V. rearranged pass PNP transistor
Connections:
- net -2.9V renamed -9.1V
- net -3V3 renamed -9V
Other:
- note added: "PA1"
- note added: "PA2"
- note added: "PA3"
- note added: "PA4"
- moved on the sheet: C11, C12, C14, C15, C4, C5, C6, C7, C8, C9, D1, D10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

Commit message: fixed minor bugs and diode choices in PA24 and updloaded almost final PA24-1. still needs to change resistor values for PA24-1
Parts:
- D1, D10, D11, D12, D13, D14, D15, D16, D17, D18, D19, D2, D20, D21, D3, D4, D5, D6, D7, D8: footprint Diode_THT:D_A-405_P12.70mm_Horizontal -> Diode_THT:D_DO-34_SOD68_P12.70mm_Horizontal
- D22, D23, D24, D25: footprint Diode_THT:D_A-405_P12.70mm_Horizontal -> Diode_THT:D_DO-35_SOD27_P12.70mm_Horizontal
Changed lines of the file:
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@@
 	(generator_version "9.0")
 	(paper "A3")
-	(text "PA3"
+	(text "PA4"
 		(exclude_from_sim no)
 		(at 128.27 254 0)
@@
 			)
 		)
-		(property "Footprint" "Diode_THT:D_A-405_P12.70mm_Horizontal"
+		(property "Footprint" "Diode_THT:D_DO-34_SOD68_P12.70mm_Horizontal"
 			(at 52.07 198.12 0)
 			(effects
@@
 			)
 		)
-		(property "Footprint" "Diode_THT:D_A-405_P12.70mm_Horizontal"
+		(property "Footprint" "Diode_THT:D_DO-34_SOD68_P12.70mm_Horizontal"
 			(at 151.13 190.5 0)
 			(effects
@@
 			)
 		)
-		(property "Footprint" "Diode_THT:D_A-405_P12.70mm_Horizontal"
+		(property "Footprint" "Diode_THT:D_DO-34_SOD68_P12.70mm_Horizontal"
 			(at 153.67 93.98 0)
 			(effects
@@
 			)
 		)
-		(property "Footprint" "Diode_THT:D_A-405_P12.70mm_Horizontal"
+		(property "Footprint" "Diode_THT:D_DO-34_SOD68_P12.70mm_Horizontal"
 			(at 346.71 190.5 0)
 			(effects
@@
 			)
 		)
-		(property "Footprint" "Diode_THT:D_A-405_P12.70mm_Horizontal"
+		(property "Footprint" "Diode_THT:D_DO-34_SOD68_P12.70mm_Horizontal"
 			(at 59.69 101.6 0)
 			(effects
@@
 			)
 		)
-		(property "Footprint" "Diode_THT:D_A-405_P12.70mm_Horizontal"
+		(property "Footprint" "Diode_THT:D_DO-34_SOD68_P12.70mm_Horizontal"
 			(at 242.57 93.98 0)
 			(effects
@@
 			)
 		)
-		(property "Footprint" "Diode_THT:D_A-405_P12.70mm_Horizontal"
+		(property "Footprint" "Diode_THT:D_DO-34_SOD68_P12.70mm_Horizontal"
 			(at 59.69 93.98 0)
 			(effects
@@
 			)
 		)
-		(property "Footprint" "Diode_THT:D_A-405_P12.70mm_Horizontal"
+		(property "Footprint" "Diode_THT:D_DO-35_SOD27_P12.70mm_Horizontal"
 			(at 64.77 190.5 0)
 			(effects
@@
 			)
 		)
-		(property "Footprint" "Diode_THT:D_A-405_P12.70mm_Horizontal"
+		(property "Footprint" "Diode_THT:D_DO-34_SOD68_P12.70mm_Horizontal"
 			(at 345.44 101.6 0)
 			(effects
@@
 			)
 		)
-		(property "Footprint" "Diode_THT:D_A-405_P12.70mm_Horizontal"
+		(property "Footprint" "Diode_THT:D_DO-34_SOD68_P12.70mm_Horizontal"
 			(at 123.19 190.5 0)
 			(effects
@@
 			)
 		)
-		(property "Footprint" "Diode_THT:D_A-405_P12.70mm_Horizontal"
+		(property "Footprint" "Diode_THT:D_DO-35_SOD27_P12.70mm_Horizontal"
 			(at 254 101.6 0)
 			(effects
@@
 			)
 		)
-		(property "Footprint" "Diode_THT:D_A-405_P12.70mm_Horizontal"
+		(property "Footprint" "Diode_THT:D_DO-34_SOD68_P12.70mm_Horizontal"
 			(at 52.07 182.88 0)
 			(effects
@@
 			)
 		)
-		(property "Footprint" "Diode_THT:D_A-405_P12.70mm_Horizontal"
+		(property "Footprint" "Diode_THT:D_DO-34_SOD68_P12.70mm_Horizontal"
 			(at 242.57 101.6 0)
 			(effects
@@
 			)
 		)
-		(property "Footprint" "Diode_THT:D_A-405_P12.70mm_Horizontal"
+		(property "Footprint" "Diode_THT:D_DO-34_SOD68_P12.70mm_Horizontal"
 			(at 128.27 95.25 0)
 			(effects
@@
 			)
 		)
-		(property "Footprint" "Diode_THT:D_A-405_P12.70mm_Horizontal"
+		(property "Footprint" "Diode_THT:D_DO-34_SOD68_P12.70mm_Horizontal"
 			(at 52.07 190.5 0)
 			(effects
@@
 			)
 		)
-		(property "Footprint" "Diode_THT:D_A-405_P12.70mm_Horizontal"
+		(property "Footprint" "Diode_THT:D_DO-35_SOD27_P12.70mm_Horizontal"
 			(at 72.39 93.98 0)
 			(effects
@@
 			)
 		)
-		(property "Footprint" "Diode_THT:D_A-405_P12.70mm_Horizontal"
+		(property "Footprint" "Diode_THT:D_DO-34_SOD68_P12.70mm_Horizontal"
 			(at 316.23 102.87 0)
 			(effects
@@
 			)
 		)
-		(property "Footprint" "Diode_THT:D_A-405_P12.70mm_Horizontal"
+		(property "Footprint" "Diode_THT:D_DO-34_SOD68_P12.70mm_Horizontal"
 			(at 320.04 191.77 0)
 			(effects
@@
 			)
 		)
-		(property "Footprint" "Diode_THT:D_A-405_P12.70mm_Horizontal"
+		(property "Footprint" "Diode_THT:D_DO-34_SOD68_P12.70mm_Horizontal"
 			(at 246.38 198.12 0)
 			(effects
@@
 			)
 		)
-		(property "Footprint" "Diode_THT:D_A-405_P12.70mm_Horizontal"
+		(property "Footprint" "Diode_THT:D_DO-34_SOD68_P12.70mm_Horizontal"
 			(at 59.69 86.36 0)
 			(effects
@@
 			)
 		)
-		(property "Footprint" "Diode_THT:D_A-405_P12.70mm_Horizontal"
+		(property "Footprint" "Diode_THT:D_DO-35_SOD27_P12.70mm_Horizontal"
 			(at 259.08 190.5 0)
 			(effects
@@
 			)
 		)
-		(property "Footprint" "Diode_THT:D_A-405_P12.70mm_Horizontal"
+		(property "Footprint" "Diode_THT:D_DO-34_SOD68_P12.70mm_Horizontal"
 			(at 246.38 190.5 0)
 			(effects
@@
 			)
 		)
-		(property "Footprint" "Diode_THT:D_A-405_P12.70mm_Horizontal"
+		(property "Footprint" "Diode_THT:D_DO-34_SOD68_P12.70mm_Horizontal"
 			(at 242.57 109.22 0)
 			(effects
@@
 			)
 		)
-		(property "Footprint" "Diode_THT:D_A-405_P12.70mm_Horizontal"
+		(property "Footprint" "Diode_THT:D_DO-34_SOD68_P12.70mm_Horizontal"
 			(at 246.38 182.88 0)
 			(effects
