File: Schematics/Reverse Engineering/PA24/PA24.kicad_sch (KiCad schematic)
At the start: 97 parts, among them J1 Conn_01x40, Q1 1N1304, Q10 PNP_G, Q11 NPN?, Q12 PNP_G, Q13 NPN?, Q14 PNP_G, Q15 NPN?, Q16 PNP_G, Q17 NPN?, Q2 PNP_G, Q3 NPN?, Q4 PNP_G, Q5 NPN?, Q6 PNP_G, Q7 NPN?, Q8 PNP_G, Q9 NPN?

Commit message: up to date versions of PA24 and PA24-1
Parts:
- D1, D10, D11, D12, D13, D14, D15, D16, D17, D18, D19, D2, D20, D21, D3, D4, D5, D6, D7, D8: footprint Diode_THT:D_A-405_P12.70mm_Horizontal -> Diode_THT:D_DO-34_SOD68_P12.70mm_Horizontal
- D22, D23, D24, D25: footprint Diode_THT:D_A-405_P12.70mm_Horizontal -> Diode_THT:D_DO-35_SOD27_P12.70mm_Horizontal
Connections:
- net -2.9V renamed -9.1V
- net -3V3 renamed -9V
Other:
- note added: "PA1"
- note added: "PA2"
- note added: "PA3"
- note added: "PA4"
- moved on the sheet: C11, C12, C14, C15, C4, C5, C6, C7, C8, C9, D1, D10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
