File: Schematics/Reverse Engineering/PA24-1/PA24-1.kicad_sch (KiCad schematic)
At the start: 113 parts, among them J1 Conn_01x40, Q1 1N1304, Q10 PNP_G, Q11 NPN?, Q12 PNP_G, Q13 NPN?, Q14 PNP_G, Q15 NPN?, Q16 PNP_G, Q17 NPN?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

Commit message: Updated resistor values in PA24-1 as they are smaller than PA24
Parts:
- R10, R14, R18, R5: value 10k -> 680
- R12, R16, R28, R8: value 39k -> 18k
- R17: value 1k -> 10k
- R20, R21, R22, R23: value 10k -> 5.1k
- R24, R25, R26, R27: value 10k -> 1k
- R29, R31, R33, R35: value 180 -> 22
Changed lines of the file:
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@@
 			)
 		)
-		(property "Value" "10k"
+		(property "Value" "1k"
 			(at 163.83 181.61 90)
 			(effects
@@
 			)
 		)
-		(property "Value" "180"
+		(property "Value" "22"
 			(at 355.6 204.47 90)
 			(effects
@@
 			)
 		)
-		(property "Value" "10k"
+		(property "Value" "680"
 			(at 316.23 115.57 90)
 			(effects
@@
 			)
 		)
-		(property "Value" "10k"
+		(property "Value" "680"
 			(at 320.04 204.47 90)
 			(effects
@@
 			)
 		)
-		(property "Value" "10k"
+		(property "Value" "5.1k"
 			(at 66.04 107.95 90)
 			(effects
@@
 			)
 		)
-		(property "Value" "10k"
+		(property "Value" "1k"
 			(at 355.6 181.61 90)
 			(effects
@@
 			)
 		)
-		(property "Value" "10k"
+		(property "Value" "5.1k"
 			(at 250.19 204.47 90)
 			(effects
@@
 			)
 		)
-		(property "Value" "1k"
+		(property "Value" "10k"
 			(at 109.22 85.09 90)
 			(effects
@@
 			)
 		)
-		(property "Value" "39k"
+		(property "Value" "18k"
 			(at 262.89 95.25 90)
 			(effects
@@
 			)
 		)
-		(property "Value" "10k"
+		(property "Value" "1k"
 			(at 163.83 85.09 90)
 			(effects
@@
 			)
 		)
-		(property "Value" "39k"
+		(property "Value" "18k"
 			(at 265.43 184.15 90)
 			(effects
@@
 			)
 		)
-		(property "Value" "39k"
+		(property "Value" "18k"
 			(at 81.28 87.63 90)
 			(effects
@@
 			)
 		)
-		(property "Value" "180"
+		(property "Value" "22"
 			(at 163.83 107.95 90)
 			(effects
@@
 			)
 		)
-		(property "Value" "180"
+		(property "Value" "22"
 			(at 163.83 204.47 90)
 			(effects
@@
 			)
 		)
-		(property "Value" "10k"
+		(property "Value" "5.1k"
 			(at 58.42 204.47 90)
 			(effects
@@
 			)
 		)
-		(property "Value" "10k"
+		(property "Value" "680"
 			(at 123.19 204.47 90)
 			(effects
@@
 			)
 		)
-		(property "Value" "10k"
+		(property "Value" "5.1k"
 			(at 247.65 115.57 90)
 			(effects
@@
 			)
 		)
-		(property "Value" "10k"
+		(property "Value" "680"
 			(at 128.27 107.95 90)
 			(effects
@@
 			)
 		)
-		(property "Value" "180"
+		(property "Value" "22"
 			(at 355.6 115.57 90)
 			(effects
@@
 			)
 		)
-		(property "Value" "39k"
+		(property "Value" "18k"
 			(at 73.66 184.15 90)
 			(effects
@@
 			)
 		)
-		(property "Value" "10k"
+		(property "Value" "1k"
 			(at 355.6 92.71 90)
 			(effects
