File: Tester/Data620-Tester-Digital/Data620-Tester-Digital.kicad_sch (KiCad schematic)
At the start: 7 parts, among them Q10 Q_NPN, Q9 Q_NPN

Commit message: fixed error in kicad design
Parts:
- removed Q10: Q_NPN, symbol Device:Q_NPN
- added Q2: Q_PNP, symbol Device:Q_PNP
- added R6: 10k, symbol Device:R
- renumbered Q9 to Q1, R36 to R1, R35 to R2, R33 to R3, R34 to R4, R37 to R5
Connections:
- net -12V: now also R6.2
- net DTL I/O: now also Q2.C, R6.1
- net GND: now also Q2.E
- net at R3.2, R4.1: now also Q2.B
