File: Schematics/Reverse Engineering/PA24-2/PA24-2.kicad_sch (KiCad schematic)
At the start: 113 parts, among them J1 Conn_01x40, Q1 2N1304, Q10 PNP_G, Q11 NPN?, Q12 PNP_G, Q13 NPN?, Q14 PNP_G, Q15 NPN?, Q16 PNP_G, Q17 NPN?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

Commit message: Revised resistor values and added images for PA24-2
Parts:
- Q11, Q15, Q3, Q7: value NPN? -> NPN2?
- R10, R14, R18, R24, R25, R26, R27, R5: value 10k -> 1k
- R12, R16, R28, R8: value 39k -> 18k
- R13, R4, R9: value 10k -> 18k
- R17: value 1k -> 18k
- R20, R21, R22, R23: value 10k -> 5.1k
Other:
- note added: "PA24-2"
- note removed: "PA24"
Changed lines of the file:
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@@
 		)
 	)
-	(text "PA24"
+	(text "PA24-2"
 		(exclude_from_sim no)
 		(at 13.97 19.05 0)
@@
 			)
 		)
-		(property "Value" "NPN?"
+		(property "Value" "NPN2?"
 			(at 115.57 190.5 90)
 			(effects
@@
 			)
 		)
-		(property "Value" "10k"
+		(property "Value" "1k"
 			(at 166.37 181.61 90)
 			(effects
@@
 			)
 		)
-		(property "Value" "10k"
+		(property "Value" "1k"
 			(at 316.23 115.57 90)
 			(effects
@@
 			)
 		)
-		(property "Value" "10k"
+		(property "Value" "1k"
 			(at 320.04 204.47 90)
 			(effects
@@
 			)
 		)
-		(property "Value" "NPN?"
+		(property "Value" "NPN2?"
 			(at 311.15 190.5 90)
 			(effects
@@
 			)
 		)
-		(property "Value" "10k"
+		(property "Value" "5.1k"
 			(at 66.04 107.95 90)
 			(effects
@@
 			)
 		)
-		(property "Value" "10k"
+		(property "Value" "1k"
 			(at 355.6 181.61 90)
 			(effects
@@
 			)
 		)
-		(property "Value" "10k"
+		(property "Value" "18k"
 			(at 101.6 184.15 90)
 			(effects
@@
 			)
 		)
-		(property "Value" "10k"
+		(property "Value" "5.1k"
 			(at 252.73 204.47 90)
 			(effects
@@
 			)
 		)
-		(property "Value" "1k"
+		(property "Value" "18k"
 			(at 111.76 85.09 90)
 			(effects
@@
 			)
 		)
-		(property "Value" "39k"
+		(property "Value" "18k"
 			(at 260.35 95.25 90)
 			(effects
@@
 			)
 		)
-		(property "Value" "10k"
+		(property "Value" "1k"
 			(at 166.37 85.09 90)
 			(effects
@@
 			)
 		)
-		(property "Value" "NPN?"
+		(property "Value" "NPN2?"
 			(at 123.19 93.98 90)
 			(effects
@@
 			)
 		)
-		(property "Value" "39k"
+		(property "Value" "18k"
 			(at 264.16 184.15 90)
 			(effects
@@
 			)
 		)
-		(property "Value" "NPN?"
+		(property "Value" "NPN2?"
 			(at 307.34 101.6 90)
 			(effects
@@
 			)
 		)
-		(property "Value" "10k"
+		(property "Value" "18k"
 			(at 293.37 95.25 90)
 			(effects
@@
 			)
 		)
-		(property "Value" "39k"
+		(property "Value" "18k"
 			(at 78.74 87.63 90)
 			(effects
@@
 			)
 		)
-		(property "Value" "10k"
+		(property "Value" "5.1k"
 			(at 58.42 204.47 90)
 			(effects
@@
 			)
 		)
-		(property "Value" "10k"
+		(property "Value" "1k"
 			(at 125.73 204.47 90)
 			(effects
@@
 			)
 		)
-		(property "Value" "10k"
+		(property "Value" "18k"
 			(at 297.18 184.15 90)
 			(effects
@@
 			)
 		)
-		(property "Value" "10k"
+		(property "Value" "5.1k"
 			(at 248.92 115.57 90)
 			(effects
@@
 			)
 		)
-		(property "Value" "10k"
+		(property "Value" "1k"
 			(at 130.81 107.95 90)
 			(effects
@@
 			)
 		)
-		(property "Value" "39k"
+		(property "Value" "18k"
 			(at 71.12 184.15 90)
 			(effects
@@
 			)
 		)
-		(property "Value" "10k"
+		(property "Value" "1k"
 			(at 355.6 92.71 90)
 			(effects
