File: Schematics/Reverse Engineering/XC31/XC31.kicad_sch (KiCad schematic)
At the start: 39 parts, among them J1 Conn_01x40, Q1 PNP, Q2 PNP, Q3 PNP, Q4 PNP, Q5 PNP, Q6 PNP, Y1 2.2MC

Commit message: Created XC31 PCB and corrected R63 to +6V instead of GND
Parts:
- added C1: 1nF, Capacitor_THT:C_Axial_L5.1mm_D3.1mm_P15.00mm_Horizontal, symbol Device:C
- added C2: 0.1uF, Capacitor_THT:C_Axial_L22.0mm_D9.5mm_P27.50mm_Horizontal, symbol Device:C
- added C3: 0.01uF, Capacitor_THT:C_Axial_L5.1mm_D3.1mm_P15.00mm_Horizontal, symbol Device:C
- C12, C13, C15, C16, C20: footprint (none) -> Capacitor_THT:C_Axial_L5.1mm_D3.1mm_P15.00mm_Horizontal
- C14, C17, C18: footprint (none) -> Capacitor_THT:C_Rect_L7.0mm_W2.0mm_P5.00mm
- C19: footprint (none) -> Capacitor_THT:C_Axial_L22.0mm_D9.5mm_P27.50mm_Horizontal
- D102, D103, D104, D105, D106, D107: footprint (none) -> Diode_THT:D_DO-34_SOD68_P12.70mm_Horizontal
- J1: footprint (none) -> Logi620:ELCO 40
- Q1, Q2, Q3, Q4, Q5, Q6: footprint (none) -> Package_TO_SOT_THT:TO-5-3; symbol Simulation_SPICE:PNP -> Transistor_BJT:Q_PNP_EBC
- R53, R54, R55, R56, R57, R58, R59, R60, R61, R62, R63, R64, R65, R66, R67, R68: footprint (none) -> Resistor_THT:R_Axial_DIN0309_L9.0mm_D3.2mm_P15.24mm_Horizontal
- Y1: footprint (none) -> Crystal:Crystal_HC51_Horizontal
Connections:
- net +6V: now also R63.1, C3.1
- net -12V: now also C1.2, C2.1
- net GND: now also Q3.1 (E), Q4.1 (E), Q5.1 (E), C1.1, C2.2, C3.2; no longer Q3.3 (E), Q4.3 (E), Q5.3 (E), R63.1
- net J1-11: now also Q1.1 (E); no longer Q1.3 (E)
- net J1-23: now also Q6.1 (E); no longer Q6.3 (E)
- net J1-7: now also Q2.1 (E); no longer Q2.3 (E)
- net at C18.1, R61.1, R62.1: now also Q4.3 (C); no longer Q4.1 (C)
- net at C12.2, R54.2: now also Q1.3 (C); no longer Q1.1 (C)
- net at C16.1, R58.1, R59.2: now also Q3.3 (C); no longer Q3.1 (C)
- net at D106.2 (A), D107.1 (K), Q6.2 (B)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: now also Q5.3 (C); no longer Q5.1 (C)
- net at C13.2, Q1.2 (B), R55.2: now also Q2.3 (C); no longer Q2.1 (C)
- net at C20.2, R68.1: now also Q6.3 (C); no longer Q6.1 (C)
- net J1-10: no longer names the net of J1.10 (Pin_10)
- net J1-12: no longer names the net of J1.12 (Pin_12)
- net J1-13: no longer names the net of J1.13 (Pin_13)
- net J1-14: no longer names the net of J1.14 (Pin_14)
- net J1-16: no longer names the net of J1.16 (Pin_16)
- net J1-17: no longer names the net of J1.17 (Pin_17)
- net J1-18: no longer names the net of J1.18 (Pin_18)
- net J1-20: no longer names the net of J1.20 (Pin_20)
- net J1-22: no longer names the net of J1.22 (Pin_22)
- net J1-24: no longer names the net of J1.24 (Pin_24)
- net J1-25: no longer names the net of J1.25 (Pin_25)
- net J1-26: no longer names the net of J1.26 (Pin_26)
- net J1-27: no longer names the net of J1.27 (Pin_27)
- net J1-28: no longer names the net of J1.28 (Pin_28)
- net J1-29: no longer names the net of J1.29 (Pin_29)
- net J1-30: no longer names the net of J1.30 (Pin_30)
- net J1-32: no longer names the net of J1.32 (Pin_32)
- net J1-33: no longer names the net of J1.33 (Pin_33)
- net J1-34: no longer names the net of J1.34 (Pin_34)
- net J1-35: no longer names the net of J1.35 (Pin_35)
- net J1-36: no longer names the net of J1.36 (Pin_36)
- net J1-38: no longer names the net of J1.38 (Pin_38)
- net J1-39: no longer names the net of J1.39 (Pin_39)
- net J1-4: no longer names the net of J1.4 (Pin_4)
- net J1-40: no longer names the net of J1.40 (Pin_40)
- net J1-5: no longer names the net of J1.5 (Pin_5)
- net J1-6: no longer names the net of J1.6 (Pin_6)
- net J1-8: no longer names the net of J1.8 (Pin_8)
- net J1-9: no longer names the net of J1.9 (Pin_9)
