File: Schematics/Reverse Engineering/ARI01/ARI01.kicad_sch (KiCad schematic)
At the start: 160 parts, among them J1 Conn_01x40, Q1 PNP, Q10 PNP, Q11 PNP, Q12 PNP, Q13 PNP, Q14 PNP, Q15 PNP, Q16 PNP, Q17 PNP, Q18 PNP, Q19 PNP, Q2 PNP, Q20 PNP, Q21 PNP, Q22 PNP, Q23 PNP, Q24 PNP, Q3 PNP, Q4 PNP, Q5 PNP, Q6 PNP, Q7 PNP, Q8 PNP, Q9 PNP

Commit message: PCB of ARI01 done. Needs to be verified
Parts:
- added R50: 5.1k, Logi620:R_Axial_DIN0207_L6.3mm_D2.5mm_P12.70mm_Horizontal, symbol Device:R
- C1, C10, C18: footprint (none) -> Capacitor_THT:C_Axial_L5.1mm_D3.1mm_P12.50mm_Horizontal
- C11, C12, C13, C14, C15, C16, C17, C2, C3, C4, C5, C6, C7, C8, C9: footprint (none) -> Capacitor_THT:C_Rect_L7.0mm_W2.0mm_P5.00mm
- D1, D19, D20, D21, D22, D35, D39, D43, D55, D57, D60: footprint (none) -> Diode_THT:D_DO-41_SOD81_P12.70mm_Horizontal
- D10, D11, D12, D13, D14, D15, D16, D17, D23, D24, D25, D26, D27, D28, D29, D30, D31, D32, D33, D34, D36, D37, D38, D40, D41, D44, D45, D46, D49, D51, D52, D53, D54, D56, D59, D61, D62, D64, D65, D67, D68, D9: footprint (none) -> Diode_THT:D_DO-34_SOD68_P12.70mm_Horizontal
- D18, D2, D3, D4, D42, D47, D48, D5, D50, D58, D6, D63, D66, D7, D8: footprint (none) -> Diode_THT:D_DO-35_SOD27_P12.70mm_Horizontal
- J1: footprint (none) -> Logi620:ELCO 40
- Q1, Q10, Q11, Q12, Q13, Q14, Q15, Q16, Q17, Q18, Q19, Q2, Q20, Q21, Q22, Q23, Q24, Q3, Q4, Q5, Q6, Q7, Q8, Q9: footprint (none) -> Package_TO_SOT_THT:TO-5-3; symbol Simulation_SPICE:PNP -> Transistor_BJT:Q_PNP_EBC
- R1, R10, R11, R12, R13, R14, R15, R16, R17, R18, R19, R2, R20, R21, R22, R23, R24, R25, R26, R27, R28, R29, R3, R30, R31, R32, R33, R34, R35, R36, R37, R38, R39, R4, R40, R42, R43, R44, R45, R46, R47, R48, R49, R5, R6, R7, R8, R9: footprint (none) -> Logi620:R_Axial_DIN0207_L6.3mm_D2.5mm_P12.70mm_Horizontal
- R41: footprint (none) -> Resistor_THT:R_Axial_DIN0309_L9.0mm_D3.2mm_P15.24mm_Horizontal
Connections:
- net -12V: now also R23.1, R50.1
- net -1V: now also Q15.1 (E), Q16.1 (E), Q17.1 (E), Q18.1 (E), Q19.1 (E), Q21.1 (E), Q22.1 (E), Q23.1 (E), Q24.1 (E); no longer Q15.3 (E), Q16.3 (E), Q17.3 (E), Q18.3 (E), Q19.3 (E), Q21.3 (E), Q22.3 (E), Q23.3 (E), Q24.3 (E)
- net GND: now also Q1.1 (E), Q10.1 (E), Q11.1 (E), Q12.1 (E), Q13.1 (E), Q14.1 (E), Q2.1 (E), Q20.1 (E), Q3.1 (E), Q4.1 (E), Q5.1 (E), Q6.1 (E), Q7.1 (E), Q8.1 (E), Q9.1 (E); no longer Q1.3 (E), Q10.3 (E), Q11.3 (E), Q12.3 (E), Q13.3 (E), Q14.3 (E), Q2.3 (E), Q20.3 (E), Q3.3 (E), Q4.3 (E), Q5.3 (E), Q6.3 (E), Q7.3 (E), Q8.3 (E), Q9.3 (E)
- net J1-16: now also Q3.3 (C); no longer Q3.1 (C)
- net J1-19: now also Q8.3 (C); no longer Q8.1 (C)
- net J1-20: now also Q13.3 (C), Q14.3 (C), Q9.3 (C); no longer Q13.1 (C), Q14.1 (C), Q9.1 (C)
- net J1-23: now also Q10.3 (C); no longer Q10.1 (C)
- net J1-25: now also Q11.3 (C); no longer Q11.1 (C)
- net J1-30: now also Q12.3 (C); no longer Q12.1 (C)
- net J1-39: now also Q1.3 (C), Q2.3 (C); no longer Q1.1 (C), Q2.1 (C)
- net at D24.2 (A), D32.2 (A), D59.2 (A)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: now also Q4.3 (C), Q5.3 (C), Q6.3 (C); no longer Q4.1 (C), Q5.1 (C), Q6.1 (C)
- net at C17.2, D66.2 (A), D67.1 (K)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: now also R50.2
- net at D26.2 (A), D29.2 (A), D55.2 (A)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: now also Q7.3 (C); no longer Q7.1 (C)
- net at D23.2 (A), D31.2 (A), R31.2: now also Q20.3 (C); no longer Q20.1 (C)
- new net: C8.2, D1.1 (K), Q15.3 (C), Q16.3 (C), Q17.3 (C), Q18.3 (C), Q19.3 (C), R12.2
- new net: C9.2, D19.1 (K), Q21.3 (C), Q22.3 (C), Q23.3 (C), Q24.3 (C), R26.2
